File: kicad_project_2/keyboard_v2.kicad_pcb (KiCad board)
At the start: 2 copper layers, 276.2 x 119.2 mm, 178 parts, among them SW1 SW_Push, U1 ATMEGA32U4, Y1 16MHz

Commit message: fix readme
Parts:
- removed REF** (x8): MountingHole_2.2mm_M2, MountingHole:MountingHole_2.2mm_M2
- C1, C2: footprint kbd:D3_TH_SMD -> kbd:D3_SMD_v2
- D69, D70, D71: footprint kbd:D3_TH -> kbd:D3_TH_SMD
- SW1: footprint Button_Switch_THT:SW_Tactile_SPST_Angled_PTS645Vx31-2LFS -> Button_Switch_THT:SW_Tactile_SPST_Angled_PTS645Vx39-2LFS
- moved C1 20.1 mm to (420.3, 6.45), turned to 0 degrees
- moved C2 16.2 mm to (420.4, 12.9), turned to 180 degrees
- moved C3 6.81 mm to (409.0, 15.8)
- moved D70 1.13 mm to (511.6, 20.8)
- moved D71 0.99 mm to (533.8, 20.5)
- moved D69 0.50 mm to (474.6, 21.4)
Routing:
- net GND: track 1132.9 -> 1102.5 mm, vias 12 -> 13
- net XTAL2: track 33.9 -> 12.9 mm
- net XTAL1: track 40.7 -> 20.8 mm
- net ROW5: track 223.8 -> 235.2 mm
- net Net-(C3-Pad1): track 12.5 -> 19.4 mm
- net Net-(D69-Pad2): track 15.3 -> 18.5 mm
- net ROW1: track 404.8 -> 407.8 mm
- net COL10: track 255.6 -> 258.2 mm
- net Net-(D70-Pad2): track 16.5 -> 18.6 mm

Commit message: fix pcb
Parts:
- added REF**: MountingHole_2.2mm_M2, MountingHole:MountingHole_2.2mm_M2, F.Cu at (469.5, -28.9)
- added REF**: MountingHole_2.2mm_M2, MountingHole:MountingHole_2.2mm_M2, F.Cu at (393.3, -29.0)
- added REF**: MountingHole_2.2mm_M2, MountingHole:MountingHole_2.2mm_M2, F.Cu at (324.1, 13.7)
- added REF**: MountingHole_2.2mm_M2, MountingHole:MountingHole_2.2mm_M2, F.Cu at (480.8, 18.7)
- added REF**: MountingHole_2.2mm_M2, MountingHole:MountingHole_2.2mm_M2, F.Cu at (566.4, 17.3)
- added REF**: MountingHole_2.2mm_M2, MountingHole:MountingHole_2.2mm_M2, F.Cu at (580.2, -70.2)
- added REF**: MountingHole_2.2mm_M2, MountingHole:MountingHole_2.2mm_M2, F.Cu at (451.0, -69.1)
- added REF**: MountingHole_2.2mm_M2, MountingHole:MountingHole_2.2mm_M2, F.Cu at (321.6, -69.1)
- moved R2 27.4 mm to (337.9, -28.6)
- moved R1 27.3 mm to (334.5, -28.7)
- moved D73 18.2 mm to (322.4, -28.0)
- moved C4 5.29 mm to (397.2, 12.3)
- moved C6 5.29 mm to (397.2, 18.2)
- moved C7 5.29 mm to (397.2, 15.1)
- moved C5 5.23 mm to (397.1, 9.21)
Routing:
- net GND: track 1102.5 -> 1344.1 mm, vias 13 -> 14
- net VCC: track 1240.8 -> 1393.3 mm, vias 9 -> 11
- net Net-(D73-Pad2): track 105.8 -> 35.7 mm, vias 1 -> 0
- net D+: track 288.1 -> 319.0 mm
- net D-: track 268.4 -> 297.8 mm
- net Net-(D73-Pad3): track 56.2 -> 45.0 mm
- net Net-(R5-Pad2): track 14.4 -> 17.5 mm
- net XTAL2: track 12.9 -> 15.7 mm
- net RESET: track 124.2 -> 127.1 mm
- net COL3: track 130.7 -> 128.0 mm

Commit message: fix pcb
Parts:
- removed REF** (x8): MountingHole_2.2mm_M2, MountingHole:MountingHole_2.2mm_M2
- added -: Val**, kbd:HOLE, F.Cu at (562.2, -69.3)
- added .: Val**, kbd:HOLE, F.Cu at (477.9, 18.0)
- added Ref**: Val**, kbd:HOLE, F.Cu at (325.6, 13.7)
- added Ref**: Val**, kbd:HOLE, F.Cu at (566.7, 16.2)
- added Ref**: Val**, kbd:HOLE, F.Cu at (444.6, -68.0)
- added Ref**: Val**, kbd:HOLE, F.Cu at (322.1, -68.5)
- F1, F2, MX1, MX10, MX11, MX12, MX13, MX14, MX15, MX16, MX17, MX18, MX19, MX2, MX20, MX21, MX22, MX23, MX24, MX25, MX26, MX27, MX28, MX29, MX3, MX30, MX31, MX32, MX33, MX34, MX35, MX36, MX37, MX38, MX39, MX4, MX40, MX41, MX42, MX43, MX44, MX45, MX46, MX47, MX48, MX49, MX5, MX50, MX51, MX52, MX53, MX54, MX55, MX56, MX57, MX58, MX59, MX6, MX60, MX61, MX62, MX63, MX64, MX65, MX66, MX67, MX68, MX69, MX7, MX70, MX8, MX9: footprint MX_Alps_Hybrid:MX-1U-NoLED -> Alps_Only:ALPS-1U
- moved C6 48.9 mm to (446.1, 15.1), turned to 270 degrees
- moved C7 46.6 mm to (443.9, 15.1), turned to 270 degrees
- moved C4 44.5 mm to (441.6, 15.0), turned to 270 degrees
- moved C5 42.5 mm to (439.2, 15.0), turned to 270 degrees
- moved C3 6.57 mm to (415.5, 16.7)
- moved Y1 6.55 mm to (426.8, 8.50)
- moved C1 6.40 mm to (426.6, 5.50)
- moved C2 6.32 mm to (426.6, 11.6)
- moved D69 5.33 mm to (469.3, 21.2)
- moved D8 2.29 mm to (479.1, -80.5)
- moved D57 2.19 mm to (428.7, -0.53)
- moved MX29 0.15 mm to (383.9, -38.1)
- moved MX30 0.13 mm to (403.0, -38.1)
- moved MX34 0.10 mm to (479.1, -38.0)
- moved MX33 0.06 mm to (460.1, -38.0)
Connections:
- U1 pad 1: (no net) -> Net-(U1-Pad1)
- U1 pad 12: (no net) -> ROW2
- U1 pad 27: (no net) -> Net-(U1-Pad27)
- U1 pad 31: (no net) -> Net-(U1-Pad31)
- U1 pad 32: (no net) -> Net-(U1-Pad32)
- U1 pad 38: ROW2 -> Net-(U1-Pad38)
- U1 pad 42: (no net) -> Net-(U1-Pad42)
- USB1 pad 3: (no net) -> Net-(USB1-Pad3)
- USB1 pad 9: (no net) -> Net-(USB1-Pad9)
- USB2 pad 3: (no net) -> Net-(USB2-Pad3)
- USB2 pad 9: (no net) -> Net-(USB2-Pad9)
Routing:
- net VCC: track 1393.3 -> 570.7 mm, vias 11 -> 5
- net GND: track 1344.1 -> 695.6 mm, vias 14 -> 11
- net D-: track 297.8 -> 339.4 mm, vias 2 -> 1
- net D+: track 319.0 -> 355.7 mm, vias 4 -> 2
- net Net-(D13-Pad2): track 36.1 -> 20.2 mm
- net XTAL2: track 15.7 -> 5.22 mm
- net COL13: track 236.5 -> 226.1 mm
- net COL9: track 246.3 -> 235.9 mm
- net COL11: track 240.8 -> 249.5 mm, vias 5 -> 4
- net Net-(D74-Pad2): track 39.9 -> 31.3 mm
- net COL10: track 258.2 -> 249.6 mm, vias 4 -> 2
- net Net-(C3-Pad1): track 19.4 -> 10.9 mm
- net COL12: track 260.7 -> 253.2 mm
- net Net-(D69-Pad2): track 18.5 -> 12.7 mm
- net ROW2: track 363.9 -> 358.3 mm
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Other:
- board size 276.2 x 119.2 mm -> 277.2 x 120.1 mm
- net class POWER: trace_width 0.5 -> 0.45

Commit message: fix pcb
Parts:
- C1, C2: footprint kbd:D3_SMD_v2 -> kbd:D3_TH_SMD
- moved F3 14.4 mm to (315.3, -16.0)
- moved R4 13.8 mm to (317.7, -16.0)
- moved R2 8.79 mm to (329.7, -31.7), turned to 270 degrees
- moved R1 8.54 mm to (329.7, -21.6)
- moved R8 5.33 mm to (441.3, 25.8)
- moved D53 2.67 mm to (334.0, -15.6)
- moved D57 2.43 mm to (426.7, -1.90)
- moved Y1 1.77 mm to (425.1, 8.55)
- moved C2 1.56 mm to (425.0, 11.6)
- moved R3 1.49 mm to (418.9, -78.7), turned to 0 degrees
- moved C1 1.42 mm to (425.2, 5.40)
- moved F4 1.37 mm to (498.1, -76.0)
- moved D28 1.32 mm to (332.4, -38.7)
- moved C3 0.58 mm to (415.5, 17.2), turned to 270 degrees
- moved F2 0.06 mm to (536.2, -80.9)
Connections:
- U1 pad 18: COL7 -> COL4
- U1 pad 19: COL8 -> COL5
- U1 pad 20: COL9 -> COL7
- U1 pad 21: COL10 -> COL8
- U1 pad 26: COL13 -> COL9
- U1 pad 28: COL4 -> COL13
- U1 pad 29: COL5 -> COL6
- U1 pad 30: COL6 -> COL10
Routing:
- net ROW1: track 404.8 -> 532.8 mm, vias 2 -> 0
- net GND: track 695.6 -> 625.4 mm, vias 11 -> 5
- net VCC: track 570.7 -> 516.4 mm
- net ROW0: track 548.8 -> 506.7 mm, vias 2 -> 4
- net Net-(D73-Pad3): track 45.0 -> 24.0 mm
- net Net-(F3-Pad2): track 40.2 -> 22.2 mm
- net COL11: track 249.5 -> 234.6 mm, vias 4 -> 2
- net Net-(R4-Pad2): track 26.6 -> 12.0 mm
- net COL4: track 131.8 -> 120.4 mm, vias 3 -> 2
- net COL5: track 122.8 -> 111.5 mm, vias 4 -> 0
- net Net-(D73-Pad2): track 35.7 -> 26.5 mm
- net COL10: track 249.6 -> 241.1 mm, vias 2 -> 0
- net COL2: track 160.7 -> 152.4 mm
- net COL13: track 226.1 -> 218.0 mm
- net XTAL1: track 17.3 -> 24.2 mm
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Other:
- outline, holes or cut-outs redrawn
- net class Default: trace_width 0.25 -> 0.2
- net class POWER: trace_width 0.45 -> 0.5
