File: kicad_project_2/keyboard_v2.kicad_pcb (KiCad board)
At the start: 2 copper layers, 277.2 x 120.1 mm, 176 parts, among them SW1 SW_Push, U1 ATMEGA32U4, Y1 16MHz

Commit message: fix parts list
Other:
- board text added: "C 1uF"
Changed lines of the file:
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@@
   )
   (dimension 277.330015 (width 0.15) (layer Dwgs.User)
-    (gr_text "277.330 mm" (at 445.636331 -178.477116 0.01859380512) (layer Dwgs.User)
+    (gr_text "277.330 mm" (at 445.65849 -110.195001 0.01859380512) (layer Dwgs.User)
       (effects (font (size 1 1) (thickness 0.15)))
     )
-    (feature1 (pts (xy 307 -90.09) (xy 306.971563 -177.718537)))
-    (feature2 (pts (xy 584.33 -90.18) (xy 584.301563 -177.808537)))
-    (crossbar (pts (xy 584.301753 -177.222116) (xy 306.971753 -177.132116)))
-    (arrow1a (pts (xy 306.971753 -177.132116) (xy 308.098066 -177.718902)))
-    (arrow1b (pts (xy 306.971753 -177.132116) (xy 308.098447 -176.546061)))
-    (arrow2a (pts (xy 584.301753 -177.222116) (xy 583.175059 -177.808171)))
-    (arrow2b (pts (xy 584.301753 -177.222116) (xy 583.17544 -176.63533)))
+    (feature1 (pts (xy 307 -90.09) (xy 306.993722 -109.436422)))
+    (feature2 (pts (xy 584.33 -90.18) (xy 584.323722 -109.526422)))
+    (crossbar (pts (xy 584.323912 -108.940001) (xy 306.993912 -108.850001)))
+    (arrow1a (pts (xy 306.993912 -108.850001) (xy 308.120225 -109.436787)))
+    (arrow1b (pts (xy 306.993912 -108.850001) (xy 308.120606 -108.263946)))
+    (arrow2a (pts (xy 584.323912 -108.940001) (xy 583.197218 -109.526056)))
+    (arrow2b (pts (xy 584.323912 -108.940001) (xy 583.197599 -108.353215)))
   )
   (gr_text "R 1k" (at 441.39 24.33) (layer B.SilkS)
@@
     (effects (font (size 0.6 0.6) (thickness 0.1)) (justify mirror))
   )
-  (gr_text "C 10uF" (at 423.99 11.41 -90) (layer B.SilkS)
+  (gr_text "C 22pF" (at 423.99 11.41 -90) (layer B.SilkS)
     (effects (font (size 0.6 0.6) (thickness 0.1)) (justify mirror))
   )
@@
     (effects (font (size 0.6 0.6) (thickness 0.1)) (justify mirror))
   )
-  (gr_text "C 10uF" (at 416.84 17.26 -90) (layer B.SilkS)
+  (gr_text "C 1uF" (at 416.84 17.26 -90) (layer B.SilkS)
     (effects (font (size 0.6 0.6) (thickness 0.1)) (justify mirror))
   )
@@
   (segment (start 308.7562 -13.0138) (end 314.06 -7.71) (width 0.5) (layer F.Cu) (net 1))
   (segment (start 314.1094 -10.4994) (end 314.1094 -7.7594) (width 0.5) (layer F.Cu) (net 1))
-  (via (at 314.06 -7.71) (size 0.762) (drill 0.4) (layers F.Cu B.Cu) (net 1) (status 1000000))
+  (via (at 314.06 -7.71) (size 0.762) (drill 0.4) (layers F.Cu B.Cu) (net 1))
   (segment (start 498.5592 -85.1114) (end 498.5592 -89.2914) (width 0.5) (layer B.Cu) (net 1))
   (segment (start 498.5592 -89.2914) (end 507.1992 -89.2914) (width 0.5) (layer B.Cu) (net 1))
